Commit message: ajout totem pizza

File: objet/totem_pizza.urdf (robot description, URDF)
Before this commit: robot physics, 4 links, 3 joints
Links:
- link bouteille: geometry collision mesh filename=pizza/pizza.obj scale=0.5 0.5 0.5; visual mesh filename=pizza/pizza.obj scale=0.5 0.5 0.5
Joints:
- joint jfixed_stuff: origin xyz=0 0 0.01 rpy=0 0 0 -> xyz=0 0 0.2 rpy=0 0 0
