Commit message: installation déco_1

File: objet/diningTable.urdf (robot description, URDF)
Before this commit: robot dinigTable, 1 links, 0 joints
Links:
- added link plantLink, mass .1; collision mesh filename=plant/eb_house_plant_01.obj scale=0.05 0.05 0.05; visual mesh filename=plant/eb_house_plant_01.obj scale=0.05 0.05 0.05
Joints:
- added joint jfixed_stuff: type fixed, parent diningTableLink, child plantLink, origin xyz=0 0 1.6 rpy=0 0 0

File: objet/plant.urdf (robot description, URDF)
Before this commit: robot table, 1 links, 0 joints
Links:
- removed link tableLink
- added link plantLink, mass .1; collision mesh filename=plant/eb_house_plant_01.obj scale=0.05 0.05 0.05; visual mesh filename=plant/eb_house_plant_01.obj scale=0.05 0.05 0.05
