Commit message: installation déco_2

File: objet/table.urdf (robot description, URDF)
Before this commit: robot table, 1 links, 0 joints
Links:
- added link tableLink2, mass .0; collision mesh filename=Table/Table_1_obj.obj scale=2.7 2.7 2.7; visual mesh filename=bar/bar3.obj scale=0.8 1 0.8
- link tableLink: geometry collision mesh filename=Table/Table_1_obj.obj scale=2.7 2.7 2.7; visual mesh filename=bar/bar.obj scale=0.5 0.4 1
Joints:
- added joint jfixed: type fixed, parent tableLink, child tableLink2, origin xyz=0 -6 0 rpy=0 0 3.14

Commit message: intégration de toutes les fonctionnalités

File: objet/table.urdf (robot description, URDF)
Before this commit: robot table, 2 links, 1 joints
Links:
- removed link tableLink2
Joints:
- removed joint jfixed
